Commit message: Problems with humble revert OS to 20.02 ubuntu

File: description/robot.urdf.xacro (robot description, xacro)
@@ -2,3 +2,6 @@
 <robot xmlns:xacro="http://www.ros.org/wiki/xacro"  name="robot">
     <xacro:include filename="robot_core.xacro"/>
+    <!-- <xacro:include filename ="gazebo_control.xacro"/> -->
+    <xacro:include filename="ros2_control.xacro"/>
+<!-- use sim time keep clocks synchronised -->
 </robot>

File: description/robot_core.xacro (robot description, xacro)
@@ -45,4 +45,5 @@
         </xacro:inertial_box>
     </link>
+    <gazebo reference="chassis"> <material> Gazebo/White </material> </gazebo>
     <!-- Left Wheel Link -->
     <joint name = "left_wheel_joint" type = "continuous">
@@ -69,4 +70,5 @@
         </xacro:inertial_cylinder>
     </link>
+    <gazebo reference="left_wheel"> <material> Gazebo/Blue </material> </gazebo>
     <!-- Right Wheel Link -->
     <joint name = "right_wheel_joint" type = "continuous">
@@ -93,4 +95,5 @@
         </xacro:inertial_cylinder>
     </link>
+        <gazebo reference="right_wheel"> <material> Gazebo/Blue </material> </gazebo>
     <!-- Caster Wheel Link -->
     <joint name="caster_wheel_joint" type = "fixed">
@@ -116,3 +119,4 @@
         </xacro:inertial_sphere>
     </link>
+        <gazebo reference="caster_wheel"> <material> Gazebo/Black </material> </gazebo>
 </robot>
