Commit message: Solving the PRoblem Every robot has

File: description/robot_core.xacro (robot description, xacro)
@@ -76,5 +76,5 @@
         <child link="right_wheel"/>
         <origin xyz ="0 -0.175 0" rpy="${pi/2} 0 0" />
-        <axis xyz="0 0 1"/>
+        <axis xyz="0 0 -1"/>
     </joint>
     <link name = "right_wheel">
@@ -119,4 +119,4 @@
         </xacro:inertial_sphere>
     </link>
-        <gazebo reference="caster_wheel"> <material> Gazebo/Black </material> </gazebo>
+        <gazebo reference="caster_wheel"> <material> Gazebo/Black </material> <mu1 value = "0.01"/> <mu2 value ="0.001"/>  </gazebo>
 </robot>

File: description/ros2_control.xacro (robot description, xacro)
@@ -24,5 +24,5 @@
     <gazebo>
         <plugin name="gazebo_ros2_control" filename="libgazebo_ros2_control.so">
-            <parameters>$(find my_bot)/config/my_controllers.yaml</parameters>
+            <parameters>/home/max/Downloads/dev-ws/my_bot/config/my_controllers.yaml</parameters>
         </plugin>
     </gazebo>
